File: hardware/pm100/pm100.kicad_sch (KiCad schematic)
At the start: 75 parts, among them J1 VCC-BATT, J10 NRST, J11 Display, J12 USART2-TX, J13 USART2-RX, J14 BOOT0, J15 GND, J16 3V3, J17 3V3, J2 VCC-ESC, J3 USB_B_Micro, J4 GND-BATT, J5 UART, J6 RECEIVER, J7 ESC, J8 SWDIO, J9 SWCLK, Q5 BSS138, Q6 BSS138, Q7 BSS138, Q8 BSS138, SW1 CLASSE, SW2 Boot0, SW3 Reset, U2 STM32L052C6Tx, U3 LD1117S50TR_SOT223, U5 LD1117S33TR_SOT223, U7 TPS2113A, U8 INA226, Y1 32.768khz, Y3 8mhz

Commit message: adicionado GND no cristal de 8mhz
Connections:
- net GND: now also Y3.2, Y3.4
Changed lines of the file:
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@@
+	)
+	(junction
+		(at 66.04 124.46)
+		(diameter 0)
+		(color 0 0 0 0)
 	)
 	(junction
@@
 	)
 	(junction
+		(at 73.66 119.38)
+		(diameter 0)
+		(color 0 0 0 0)
+	)
+	(junction
 		(at 246.38 83.82)
 		(diameter 0)
@@
 	(wire
 		(pts
+			(xy 66.04 119.38) (xy 66.04 124.46)
+		)
+		(stroke
+			(width 0)
+			(type default)
+		)
+	)
+	(wire
+		(pts
 			(xy 76.2 109.22) (xy 60.96 109.22)
 		)
@@
 	(wire
 		(pts
+			(xy 73.66 119.38) (xy 73.66 124.46)
+		)
+		(stroke
+			(width 0)
+			(type default)
+		)
+	)
+	(wire
+		(pts
 			(xy 121.92 116.84) (xy 135.89 116.84)
 		)
@@
 		)
 		(stroke
+			(width 0)
+			(type default)
+		)
+	)
+	(wire
+		(pts
+			(xy 73.66 119.38) (xy 66.04 119.38)
+		)
+		(stroke

Commit message: usando Xiao Ble
Connections:
- net 2-rx: now reaches J13.1 (Pin_1), U2.13 (PA3)
- net swclk: now reaches J9.1 (Pin_1), U2.37 (PA14)
- net 2-tx: now reaches J12.1 (Pin_1), U2.12 (PA2)
- net swdio: now reaches J8.1 (Pin_1), U2.34 (PA13)
- net boot0: now reaches J14.1 (Pin_1), R12.2, SW2.2, U2.44 (BOOT0)
- net RST: now reaches C6.1, J10.1 (Pin_1), SW3.1, U2.7 (NRST)
Changed lines of the file:
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@@
 (kicad_sch
-	(version 20231120)
+	(version 20250114)
 	(generator "eeschema")
-	(generator_version "8.0")
+	(generator_version "9.0")
 	(paper "A4")
 	(junction
@@
 		)
 	)
+	(label "2-rx"
+		(at 129.54 121.92 0)
+		(effects
+			(font
+				(size 1.27 1.27)
+			)
+			(justify left bottom)
+		)
+	)
+	(label "3v3"
+		(at 57.15 116.84 0)
+		(effects
+			(font
+				(size 1.27 1.27)
+			)
+			(justify left bottom)
+		)
+	)
+	(label "swdio"
+		(at 128.27 144.78 0)
+		(effects
+			(font
+				(size 1.27 1.27)
+			)
+			(justify left bottom)
+		)
+	)
+	(label "boot0"
+		(at 77.47 116.84 0)
+		(effects
+			(font
+				(size 1.27 1.27)
+			)
+			(justify left bottom)
+		)
+	)
+	(label "swclk"
+		(at 128.27 147.32 0)
+		(effects
+			(font
+				(size 1.27 1.27)
+			)
+			(justify left bottom)
+		)
+	)
+	(label "2-tx"
+		(at 129.54 116.84 0)
+		(effects
+			(font
+				(size 1.27 1.27)
+			)
+			(justify left bottom)
+		)
+	)
+	(label "RST"
+		(at 76.2 106.68 0)
+		(effects
+			(font
+				(size 1.27 1.27)
+			)
+			(justify left bottom)
+		)
+	)
 	(global_label "AN-CLASSE"
 		(shape input)
@@
 		)
 	)
+	(embedded_fonts no)
 )
