File: hardware/pm100-xiao/pm100.kicad_sch (KiCad schematic)
At the start: 42 parts, among them J1 VCC-BATT, J10 NRST, J2 VCC-ESC, J4 GND-BATT, J5 UART, J6 RECEIVER, J7 ESC, J8 SWDIO, J9 SWCLK, Q5 BSS138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

Commit message: ajustando pinagem LED RGBA
Connections:
- net GND: now also D2.2 (VSS); no longer D2.3 (VSS)
- net LED: now also D2.3 (DIN); no longer D2.4 (DIN)
- net at C7.1, D3.1 (K): now also D2.4 (VDD); no longer D2.1 (VDD)
