File: hardware/pm100-xiao/pm100.kicad_pcb (KiCad board)
At the start: 2 copper layers, 39.1 x 68.6 mm, 42 parts, among them J1 VCC-BATT, J10 NRST, J2 VCC-ESC, J4 GND-BATT, J5 UART, J6 RECEIVER, J7 ESC, J8 SWDIO, J9 SWCLK, Q5 BSS138, Q6 BSS138, Q7 BSS138, Q8 BSS138, SW1 CLASSE, SW3 Reset, U3 LD1117S50TR_SOT223, U8 INA226

Commit message: atualizando fonte e adicionado entrada auxiliar para desligar controle
Parts:
- removed J10: NRST, TestPoint:TestPoint_Pad_D2.0mm
- removed J8: SWDIO, TestPoint:TestPoint_Pad_D2.0mm
- removed J9: SWCLK, TestPoint:TestPoint_Pad_D2.0mm
- removed SW1: CLASSE, Button_Switch_SMD:SW_SP3T_PCM13
- removed SW3: Reset, Button_Switch_SMD:SW_SPST_B3U-3100P-B
- removed U3: LD1117S50TR_SOT223, Package_TO_SOT_SMD:SOT-223-3_TabPin2
- added C4: 0.1u, Capacitor_SMD:C_0805_2012Metric, F.Cu at (130.4, 46.5)
- added L1: Hcnr6045-220m, Inductor_SMD:L_Bourns_SRN6045TA, F.Cu at (124.1, 48.7)
- added Q9: BSS138, Package_TO_SOT_SMD:SOT-23, F.Cu at (127.7, 54.7)
- added R12: 100k, Resistor_SMD:R_0603_1608Metric, F.Cu at (118.1, 51.2)
- added R13: 100k, Resistor_SMD:R_0603_1608Metric, F.Cu at (118.1, 53.8)
- added R14: 18k, Resistor_SMD:R_0603_1608Metric, F.Cu at (118.1, 56.3)
- added U2: LMR16006YQ5, Package_TO_SOT_SMD:SOT-23-6, F.Cu at (122.7, 54.9)
- C3: renamed from C4; value 0.1u -> 4.7u; footprint Capacitor_SMD:C_0603_1608Metric -> Capacitor_SMD:C_0805_2012Metric
- C6: value 0.1u -> 10u; footprint Capacitor_SMD:C_0603_1608Metric -> Capacitor_SMD:C_0805_2012Metric
- moved R6 28.8 mm to (118.1, 46.2)
- moved R7 26.4 mm to (118.1, 48.7), turned to 0 degrees
- moved C6 23.2 mm to (130.4, 49.5), turned to 0 degrees
Connections:
- C5 pad 1: Net-(D4-A) -> +5V
- C6 pad 1: /RST -> Net-(D4-K)
- C6 pad 2: GND -> Net-(U2-CB)
- D4 pad 1: +5V -> Net-(D4-K)
- D4 pad 2: Net-(D4-A) -> GND
- R6 pad 1: GND -> PWM-RECEIVER-2
- R6 pad 2: Net-(R6-Pad2) -> +5V
- R7 pad 1: +3V3 -> PWM-INPUT-2
- R7 pad 2: Net-(R6-Pad2) -> +3V3
- U1 pad 11: LED -> unconnected-(U1-MOSI/P1.15-Pad11)
- U1 pad 15: Net-(J9-Pin_1) -> unconnected-(U1-CLK-Pad15)
- U1 pad 17: /RST -> unconnected-(U1-RST-Pad17)
- U1 pad 18: Net-(J8-Pin_1) -> LED
- U1 pad 2: AN-CLASSE -> PWM-INPUT-2
Routing:
- net unconnected-(U1-RST-Pad17): track 0.00 -> 33.5 mm, vias 0 -> 1
- net /RST: track 33.5 -> 0.00 mm, vias 1 -> 0
- net AN-CLASSE: track 32.7 -> 0.00 mm, vias 1 -> 0
- net (no net): track 0.00 -> 29.4 mm
- net Net-(D4-A): track 23.8 -> 0.00 mm, vias 1 -> 0
- net Net-(J9-Pin_1): track 23.2 -> 0.00 mm, vias 2 -> 0
- net Net-(J8-Pin_1): track 16.6 -> 0.00 mm
- net +3V3: track 87.7 -> 77.2 mm, vias 4 -> 3
- net Net-(R6-Pad2): track 5.58 -> 0.00 mm
- net LED: track 43.5 -> 39.4 mm
- net unconnected-(U1-MOSI/P1.15-Pad11): track 0.00 -> 3.59 mm
- net GND: vias 11 -> 12

Commit message: rev4 projeto eletronico
Parts:
- removed J1: VCC-BATT, footprints:HV_CONN_01x01_pad_6.2x12mm
- removed J4: GND-BATT, footprints:HV_CONN_01x01_pad_6.2x12mm
- added J3: HV-ESC, Connector_AMASS:AMASS_XT60PW-F_1x02_P7.20mm_Horizontal, F.Cu at (219.3, 54.6)
- added J8: SAFETY, pm100:smd-pwm-3-Wire, B.Cu at (221.7, 79.0)
- C1, C2, Q9, R1, R24, R25, R6, R7, U8: moved to B.Cu
- C3, C5, D1, D2, U1: moved to F.Cu
- D4: value D_Schottky -> SS18
- J2: value VCC-ESC -> HV-BATTERY; footprint footprints:HV_CONN_01x01_pad_6.2x12mm -> Connector_AMASS:AMASS_XT60IPW-M_1x03_P7.20mm_Horizontal
- J5: footprint Connector_JST:JST_XH_S4B-XH-A-1_1x04_P2.50mm_Horizontal -> Connector_Hirose:Hirose_DF13-04P-1.25DS_1x04_P1.25mm_Horizontal; moved to F.Cu
- J6, J7: footprint Sigma Footprints:SolderWire_SMD_3 -> pm100:smd-pwm-3-Wire
- moved R13 118.4 mm to (235.5, 69.3), turned to -90 degrees
- moved R14 116.6 mm to (233.9, 69.3), turned to -90 degrees
- moved R12 115.4 mm to (233.0, 62.0), turned to -90 degrees
- moved L1 113.9 mm to (237.0, 64.2), turned to -90 degrees
- moved U2 109.8 mm to (232.0, 65.4), turned to 90 degrees
- moved R6 105.6 mm to (220.5, 72.1), turned to 90 degrees
- moved R7 103.0 mm to (217.7, 75.2), turned to -90 degrees
- moved C6 102.6 mm to (231.1, 68.6)
- moved C4 102.0 mm to (231.2, 61.8), turned to -90 degrees
- moved J5 97.4 mm to (238.1, 85.7), turned to 180 degrees
- moved R8 95.1 mm to (237.2, 83.6)
- moved Q9 94.9 mm to (220.4, 75.2)
- moved Q7 93.9 mm to (238.3, 80.8), turned to -90 degrees
- moved R9 92.4 mm to (238.3, 78.0), turned to 0 degrees
- moved R11 88.0 mm to (234.2, 83.6), turned to 0 degrees
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Connections:
- J2 pad 1: Net-(J2-Pin_1) -> GND
- R1 pad 1: +BATT -> Net-(J3-Pin_2)
- R1 pad 4: Net-(J2-Pin_1) -> +BATT
- R24 pad 1: Net-(R1-Pad2) -> Net-(R1-Pad3)
- R25 pad 1: Net-(R1-Pad3) -> Net-(R1-Pad2)
- U1 pad 11: unconnected-(U1-MOSI/P1.15-Pad11) -> LED
- U1 pad 18: LED -> unconnected-(U1-DIO-Pad18)
Routing:
- net unconnected-(U1-RST-Pad17): track 33.5 -> 0.00 mm, vias 1 -> 0
- net PWM-OUTPUT: track 53.5 -> 22.1 mm, vias 2 -> 1
- net (no net): track 29.4 -> 0.00 mm
- net LED: track 39.4 -> 14.2 mm, vias 2 -> 0
- net PWM-INPUT-2: track 0.00 -> 24.6 mm, vias 0 -> 1
- net +BATT: track 23.7 -> 47.2 mm, vias 1 -> 0
- net +5V: track 87.9 -> 68.5 mm
- net +3V3: track 77.2 -> 57.9 mm, vias 3 -> 7
- net Net-(D4-K): track 0.00 -> 17.1 mm, vias 0 -> 3
- net GND: track 38.5 -> 21.5 mm, vias 12 -> 2
- net Net-(J3-Pin_2): track 0.00 -> 12.8 mm
- net PWM-INPUT: track 46.4 -> 33.9 mm, vias 2 -> 1
- net UART_{0}-TX: track 23.2 -> 11.3 mm, vias 1 -> 0
- net I2C-SDA: track 20.6 -> 9.06 mm
- net /Tx: track 15.4 -> 7.86 mm, vias 0 -> 2
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- removed copper zone on F.Cu, net +BATT
- removed copper zone on B.Cu, net GND
- removed copper zone on F.Cu, net GND
Other:
- board size 39.1 x 68.6 mm -> 32.2 x 44 mm
- board text added: "36VDC 90A"
- board text added: "9600bps"
- board text added: "BYPASS"
- board text added: "INPUT"
- board text added: "REV4 260926"
- board text added: "RX"
- board text added: "TX"
- board text added: "VCC"
- board text removed: "GND VCOM RX TX"
- board text removed: "RECV"
- board text removed: "REG MICRO ADV"
- board text removed: "Sinal"

Commit message: bug logs não salvos, revisão do hardware pronta para produção
Parts:
- removed H1: MountingHole, MountingHole:MountingHole_3.2mm_M3_ISO7380
- moved C1 88.0 mm to (136.4, 90.6)
- moved C3 88.0 mm to (146.4, 78.3)
- moved D1 88.0 mm to (136.4, 80.0)
- moved D4 88.0 mm to (142.3, 83.3)
- moved J2 88.0 mm to (142.8, 74.2)
- moved J5 88.0 mm to (152.3, 105.3)
- moved J7 88.0 mm to (150.6, 98.6)
- moved L1 88.0 mm to (151.2, 83.8)
- moved Q5 88.0 mm to (128.7, 95.0)
- moved Q6 88.0 mm to (151.7, 94.3)
- moved Q7 88.0 mm to (152.4, 100.4)
- moved Q8 88.0 mm to (148.6, 100.4)
- moved R1 88.0 mm to (138.4, 80.4)
- moved R10 88.0 mm to (148.6, 97.6)
- moved R12 88.0 mm to (147.2, 81.6)
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Routing:
- net GND: track 21.5 -> 50.7 mm, vias 2 -> 7
- net LED: track 14.2 -> 31.5 mm
- net Net-(D2-VDD): track 9.63 -> 12.5 mm
- net Net-(U2-~{SHDN}): track 0.00 -> 1.45 mm
- added copper zone on B.Cu, net GND
- added copper zone on F.Cu, net GND
